Commit message: fix end effector joint frame origin to the end of arm2

File: robot_data/2link_robot.urdf (robot description, URDF)
Before this commit: robot 2link_robot, 4 links, 3 joints
Links:
- link arm1: geometry collision box size=1 .05 .05; visual box size=1 .05 .05
- link arm2: geometry collision box size=1 .05 .05; visual box size=1 .05 .05
Joints:
- joint ee_joint: origin xyz=0 0 0.05 rpy=0 0 0 -> xyz=1 0 0.05 rpy=0 0 0
