Commit message: add panda description

File: robot_data/panda_description/urdf/panda_no_gripper_simple_collision.urdf (robot description, URDF)
Before this commit: robot panda, 9 links, 8 joints
Links:
- link panda_link0: geometry collision cylinder length=0.03 radius=0.06; collision sphere radius=0.06
- link panda_link1: geometry collision cylinder length=0.2830 radius=0.06; collision sphere radius=0.06
- link panda_link2: geometry collision cylinder length=0.12 radius=0.06; collision sphere radius=0.06
- link panda_link3: geometry collision cylinder length=0.15 radius=0.06; collision sphere radius=0.06
- link panda_link4: geometry collision cylinder length=0.12 radius=0.06; collision sphere radius=0.06
- link panda_link5: geometry collision cylinder length=0.1 radius=0.06; collision cylinder length=0.14 radius=0.025
- link panda_link6: geometry collision cylinder length=0.08 radius=0.05; collision sphere radius=0.05
- link panda_link7: geometry collision cylinder length=0.14 radius=0.04; collision sphere radius=0.04

File: robot_data/panda_description/urdf/panda_simple_collision.urdf (robot description, URDF)
Before this commit: robot panda, 12 links, 11 joints
Links:
- link panda_hand: geometry collision cylinder length=0.1 radius=0.02; collision cylinder length=0.1 radius=0.04
- link panda_leftfinger: geometry visual mesh filename=meshes/visual/finger.dae
- link panda_link0: geometry collision cylinder length=0.03 radius=0.06; collision sphere radius=0.06
- link panda_link1: geometry collision cylinder length=0.2830 radius=0.06; collision sphere radius=0.06
- link panda_link2: geometry collision cylinder length=0.12 radius=0.06; collision sphere radius=0.06
- link panda_link3: geometry collision cylinder length=0.15 radius=0.06; collision sphere radius=0.06
- link panda_link4: geometry collision cylinder length=0.12 radius=0.06; collision sphere radius=0.06
- link panda_link5: geometry collision cylinder length=0.1 radius=0.06; collision cylinder length=0.14 radius=0.025
- link panda_link6: geometry collision cylinder length=0.08 radius=0.05; collision sphere radius=0.05
- link panda_link7: geometry collision cylinder length=0.14 radius=0.04; collision sphere radius=0.04
- link panda_rightfinger: geometry visual mesh filename=meshes/visual/finger.dae
